Commit message: Rviz showing only base link

File: src/rviz_sim/urdf/model_core.urdf.xacro (robot description, xacro)
@@ -2,4 +2,5 @@
 <robot name="myfirst" xmlns:xacro="http://www.ros.org/wiki/xacro">
     <xacro:include filename="wings.xacro"/>
+    <link name="world"/>
     <joint name="base_joint" type="fixed">
         <parent link="world"/>
