Commit message: Gazebo and Rviz now showing robot transformation
Problem: ros2_control uses the joint_state_broadcaster topic to publish the joint_state information. When the joint_state_publisher was active, both the jsp and jsb published on the joint_state topic causing a cyclic graph between jsp -> joint_state -> robot_state_publisher -> robot_description. This caused Rviz to only show the jsp output

Fix: remove the joint_state_publisher node. Ensure that all the non-fixed joints are in the ros2_control tag.

File: src/rviz_sim/urdf/controller.xacro (robot description, xacro)
@@ -12,5 +12,19 @@
 			<state_interface name="velocity"/>
 		</joint>
+		<joint name="right_rotating_arm_joint">
+			<command_interface name="position">
+				<param name="initial_value">0.0</param>
+			</command_interface>
+			<state_interface name="position"/>
+			<state_interface name="velocity"/>
+		</joint>
 		<joint name="left_slider_joint">
+			<command_interface name="position">
+				<param name="initial_value">0.0</param>
+			</command_interface>
+			<state_interface name="position"/>
+			<state_interface name="velocity"/>
+		</joint>
+		<joint name="left_rotating_arm_joint">
 			<command_interface name="position">
 				<param name="initial_value">0.0</param>
